File: li-ion-backup-board/li-ion-backup.sch (KiCad schematic (older format))
At the start: 70 parts

Commit message: update components value
Parts:
- removed R?: R, Resistor_SMD:R_0805_2012Metric, symbol Device:R
- removed R?: 0R1, Resistor_SMD:R_0805_2012Metric, symbol Device:R
- added F?: Fuse, e-Power:FUSE_1206_3216Metric, symbol Device:Fuse
- added R?: 0R1, Resistor_SMD:R_1206_3216Metric, symbol Device:R
- C?: value C -> 1uF; LCSC (none) -> C28323
- C? (x4): value C -> 10nF; LCSC (none) -> C1710
- C? (x6): value CP -> 220uF; LCSC (none) -> C311611; Voltage  (none) -> 35V
- C? (x7): value C -> 100nF; LCSC (none) -> C49678; Voltage  (none) -> 50V
- C? (x2): value C -> 10uF; LCSC (none) -> C15850; Voltage  (none) -> 25V
- C?: LCSC (none) -> C49678; Voltage  (none) -> 50V
- D?: value GRN -> GREEN
- L? (x4): LCSC (none) -> C151872
- L?: value 10uH -> 15uH; LCSC (none) -> C151872
- R?: value R -> 2.2R; LCSC (none) -> C17521
- R? (x2): value R -> ADJ
- R?: value R -> 12K; LCSC (none) -> C17444
- R?: value R -> 3K9; LCSC (none) -> C17614
- R?: LCSC (none) -> C17379
- R?: footprint Resistor_SMD:R_0805_2012Metric -> Resistor_SMD:R_1206_3216Metric; LCSC (none) -> C25334
- R? (x7): LCSC (none) -> C17513
- R?: LCSC (none) -> C17408
- R? (x2): LCSC (none) -> C17414
- R?: LCSC (none) -> C25826
- R? (x2): LCSC (none) -> C17477
- U?: LCSC (none) -> C99046
Connections:
- net +5V: now also R?.2
- net at C?.1, C?.1, L?.1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: now also R?.1
- net at C?.1, C?.2, D?.2 (A)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: now also R?.1
- net at D?.1 (K), D?.2 (A), R?.1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: now also F?.1; no longer J?.2 (Pin_2)
- new net: F?.2, J?.2 (Pin_2)
Other:
- note removed: "1A de carregamento"
- note removed: "2A de saída"
- note removed: "Funcionalidade de medição de temperatura (?)"
- moved on the sheet: C?, J?, R?
